File: bus blaster adapter.kicad_pcb (KiCad board)
At the start: 2 copper layers, 50 x 50 mm, 72 parts, among them P101 CONN_02X10, P102 CONN_02X10

Commit message: Layout work, could probably use double checking...
Parts:
- added P103: CONN_02X05, header_1:10pin_1.27pitch, F.Cu at (102.4, 108.5)
- added REF**: Symbol_OSHW-Logo_CopperTop, Symbols:Symbol_OSHW-Logo_CopperTop, F.Cu at (144.0, 108.0)
- moved JP169 2.46 mm to (106.0, 108.0)
- moved P101 2.40 mm to (143.1, 114.5)
- moved JP101 2.06 mm to (106.5, 142.0)
- moved JP102 2.06 mm to (111.0, 142.0)
- moved JP170 2.00 mm to (103.0, 142.0)
- turned JP150 to 0 degrees
Routing:
- net GND: track 268.3 -> 223.4 mm
- net Net-(JP153-Pad2): track 39.3 -> 53.7 mm
- net Net-(JP110-Pad2): track 41.7 -> 56.1 mm
- net Net-(JP117-Pad2): track 42.8 -> 56.3 mm, vias 0 -> 1
- net Net-(JP123-Pad2): track 40.8 -> 53.7 mm, vias 0 -> 1
- net Net-(JP160-Pad2): track 36.3 -> 49.2 mm
- net Net-(JP128-Pad2): track 40.7 -> 52.3 mm, vias 0 -> 1
- net Net-(JP147-Pad2): track 41.0 -> 51.2 mm, vias 0 -> 1
- net Net-(JP142-Pad2): track 37.6 -> 46.7 mm, vias 0 -> 1
- net /VTREF: track 126.1 -> 118.1 mm, vias 9 -> 8
- net /TDI: track 105.8 -> 99.0 mm
- net /TSRST: track 106.1 -> 100.1 mm, vias 8 -> 7
- net Net-(JP133-Pad2): track 50.0 -> 55.6 mm
- net Net-(JP139-Pad2): track 19.5 -> 23.7 mm
- net /TDO: track 85.6 -> 81.4 mm
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Other:
- board size 50 x 50 mm -> 50 x 43 mm
- board text added: "14 20 10 10 10 10 14 14"
- board text added: ">or"
- board text added: "A"
- board text added: "B"
- board text added: "Blackfin Compact TI Tag Connect Maxim MAXQ AVR ByteBlaster MIPS EJTAG ARM-14"
- board text added: "C"
- board text added: "C A D E A B F H A B G H A B H A B I A B J"
- board text added: "Configured For:"
- board text added: "D"
- board text added: "E"
- board text added: "F"
- board text added: "G"
- board text added: "H"
- board text added: "Host"
- board text added: "Ian Rees - July 2016 - v1"
- board text added: "J"
- board text added: "Jumper Sections"
- board text added: "TI EMU0"
- board text added: "TI EMU1"
- board text added: "Target"
- board text added: "Target Pins Used"
- board text added: "github.com/ianrrees/busblaster-adapter"
- board text removed: "ARM-14"
- board text removed: "AVR"
- board text removed: "Blackfin"
- board text removed: "ByteBlaster"
- board text removed: "Compact TI 20-pin"
- board text removed: "MAXQ"
- board text removed: "MIPS EJTAG"
- board text removed: "Tag Connect"

Commit message: Copper pours!
Routing:
- added copper zone on B.Cu, net GND
- added copper zone on F.Cu, net GND
Changed lines of the file:
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@@
     (area 97.924999 103.924999 148.075001 147.075001)
     (thickness 1.6)
-    (drawings 58)
+    (drawings 60)
     (tracks 876)
     (zones 0)
@@
     (zone_45_only no)
     (trace_min 0.2)
-    (segment_width 0.2)
+    (segment_width 0.15)
     (edge_width 0.15)
     (via_size 0.6)
@@
     (fp_line (start 0.35052 0.89916) (end 0.7493 1.89992) (layer F.Cu) (width 0.381))
   )
+  (gr_line (start 101.8 131) (end 105.6 131) (layer F.SilkS) (width 0.15))
+  (gr_line (start 101.8 126) (end 105.6 126) (layer F.SilkS) (width 0.15))
   (gr_text "Configured\nFor:" (at 129 134) (layer F.SilkS)
     (effects (font (size 1.5 1.5) (thickness 0.3)) (justify right))
@@
     (effects (font (size 1.5 1.5) (thickness 0.3)) (justify left mirror))
   )
-  (gr_text "Blackfin\nCompact TI\nTag Connect\nMaxim MAXQ\nAVR\nByteBlaster\nMIPS EJTAG\nARM-14" (at 128 107 90) (layer B.SilkS)
-    (effects (font (size 1.5 1.5) (thickness 0.3)) (justify left mirror))
+  (gr_text "Blackfin\nCompact TI\nTag Connect\nMaxim MAXQ\nAVR\nByteBlaster\nMIPS EJTAG\nARM-14" (at 128 122.2 90) (layer B.SilkS)
+    (effects (font (size 1.5 1.5) (thickness 0.3)) (justify right mirror))
   )
   (gr_arc (start 145 107) (end 145 104) (angle 90) (layer Edge.Cuts) (width 0.15))
@@
       )
     )
+  )
+  (zone (net 1) (net_name GND) (layer F.Cu) (hatch edge 0.508)
+    (connect_pads (clearance 0.508))
+    (min_thickness 0.254)
+    (fill yes (arc_segments 32) (thermal_gap 0.508) (thermal_bridge_width 0.508))
+    (polygon
+      (pts
+        (xy 98 104) (xy 148 104) (xy 148 147) (xy 98 147)
+      )
+    )
+  )
+  (zone (net 1) (net_name GND) (layer B.Cu) (hatch edge 0.508)
+    (connect_pads (clearance 0.508))
+    (min_thickness 0.254)
+    (fill yes (arc_segments 16) (thermal_gap 0.508) (thermal_bridge_width 0.508))
+    (polygon
+      (pts
+        (xy 98 104) (xy 148 104) (xy 148 147) (xy 98 147)
+      )
+    )

Commit message: Tidy up, as much as one can call it that...
Parts:
- turned JP139 to 0 degrees
Routing:
- net GND: track 223.4 -> 271.9 mm, vias 15 -> 16
- net /VTREF: track 118.1 -> 136.9 mm, vias 8 -> 7
- net /TRST: track 96.3 -> 81.1 mm, vias 7 -> 6
- net /TSRST: track 100.1 -> 90.4 mm
- net /TCK: track 70.8 -> 79.7 mm
- net /TDI: track 99.0 -> 94.5 mm
- net /TDO: track 81.4 -> 84.8 mm, vias 7 -> 5
- net Net-(JP139-Pad2): track 23.7 -> 26.1 mm
- net Net-(JP133-Pad2): track 55.6 -> 54.2 mm
- net /TMS: track 59.1 -> 58.5 mm
Other:
- board text added: "Ian Rees - July 2016 - Dunedin NZ"
- board text added: "V1"
- board text removed: "Ian Rees - July 2016 - v1"
